File: TPS62133/KiCad Project Files/TPS62133.kicad_sch (KiCad schematic)
At the start: 10 parts, among them J1 Conn_01x03, J2 Conn_01x02, U1 TPS62133

Commit message: updated TPS62133
Parts:
- C2: footprint Capacitor_SMD:C_0603_1608Metric -> Capacitor_SMD:C_0805_2012Metric_Pad1.15x1.40mm_HandSolder
- R1: footprint Resistor_SMD:R_0603_1608Metric -> Resistor_SMD:R_0805_2012Metric_Pad1.15x1.40mm_HandSolder
Connections:
- net Vin renamed +12V
Other:
- company: (none) -> SlugCharge
- title: (none) -> TPS62133 Charging Circuit
Changed lines of the file:
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@@
   (page 1 1)
   (paper "A4")
+  (title_block
+    (title "TPS62133 Charging Circuit")
+    (date "2020-05-20")
+    (rev "1.0")
+    (company "SlugCharge")
+    (comment 1 "Engineer: Aditya Sehgal")
+  )
+  (junction (at 111.76 93.98))
   (junction (at 115.57 93.98))
   (junction (at 115.57 102.87))
@@
   (junction (at 167.64 102.87))
   (junction (at 167.64 121.92))
+  (junction (at 181.61 100.33))
   (wire (pts (xy 107.95 106.68) (xy 111.76 106.68)))
   (wire (pts (xy 107.95 111.76) (xy 111.76 111.76)))
@@
     )
   )
+  (symbol (lib_id "power:+12V") (at 111.76 93.98 0) (unit 1)
+    (property "Reference" "#PWR?" (id 0) (at 111.76 97.79 0)
+      (effects (font (size 1.27 1.27)) hide)
+    )
+    (property "Value" "+12V" (id 1) (at 112.1283 89.6556 0))
+    (property "Footprint" "" (id 2) (at 111.76 93.98 0)
+      (effects (font (size 1.27 1.27)) hide)
+    )
+    (property "Datasheet" "" (id 3) (at 111.76 93.98 0)
+      (effects (font (size 1.27 1.27)) hide)
+    )
+  )
+  (symbol (lib_id "power:+5V") (at 181.61 100.33 0) (unit 1)
+    (property "Reference" "#PWR?" (id 0) (at 181.61 104.14 0)
+      (effects (font (size 1.27 1.27)) hide)
+    )
+    (property "Value" "+5V" (id 1) (at 181.9783 96.0056 0))
+    (property "Footprint" "" (id 2) (at 181.61 100.33 0)
+      (effects (font (size 1.27 1.27)) hide)
+    )
+    (property "Datasheet" "" (id 3) (at 181.61 100.33 0)
+      (effects (font (size 1.27 1.27)) hide)
+    )
+  )
   (symbol (lib_id "power:GNDREF") (at 143.51 121.92 0) (unit 1)
     (property "Reference" "#PWR0101" (id 0) (at 143.51 128.27 0)
@@
     (property "Reference" "R1" (id 0) (at 162.56 96.52 90))
     (property "Value" "100K" (id 1) (at 162.56 97.79 90))
-    (property "Footprint" "Resistor_SMD:R_0603_1608Metric" (id 2) (at 162.56 100.33 0)
+    (property "Footprint" "Resistor_SMD:R_0805_2012Metric_Pad1.15x1.40mm_HandSolder" (id 2) (at 162.56 100.33 0)
       (effects (font (size 1.27 1.27)) hide)
     )
@@
     )
   )
-  (symbol (lib_id "Device:C_Small") (at 123.19 109.22 0) (unit 1)
+  (symbol (lib_name "Device:C_Small_3") (lib_id "Device:C_Small") (at 123.19 109.22 0) (unit 1)
     (property "Reference" "C2" (id 0) (at 125.73 107.95 0)
       (effects (font (size 1.27 1.27)) (justify left))
@@
       (effects (font (size 1.27 1.27)) (justify left))
     )
-    (property "Footprint" "Capacitor_SMD:C_0603_1608Metric" (id 2) (at 123.19 109.22 0)
+    (property "Footprint" "Capacitor_SMD:C_0805_2012Metric_Pad1.15x1.40mm_HandSolder" (id 2) (at 123.19 109.22 0)
       (effects (font (size 1.27 1.27)) hide)
     )
@@
     (path "/b1974ded-7503-4572-98ec-212e2de9c175" (reference "#PWR0102") (unit 1))
     (path "/e6e0f3f0-fd5f-4289-82ff-473cdf8db748" (reference "#PWR0103") (unit 1))
+    (path "/4d96844f-beed-477a-a0a1-af7d3701838a" (reference "#PWR?") (unit 1))
+    (path "/ba3fa7c4-79af-4e49-a2b2-a83c0eacce2c" (reference "#PWR?") (unit 1))
     (path "/d9dfa453-db02-4981-8156-77a74b3e0e1a" (reference "C1") (unit 1))
     (path "/7d1fd7d5-2b9c-43ad-9d61-276daf86cc0c" (reference "C2") (unit 1))
