File: SlugCharge Daughterboard/KiCad Project FIles/Locker1.kicad_sch (KiCad schematic)
At the start: 43 parts, among them J1 Locker in, J10 Locker out, J2 Conn_01x04, J3 Unreg 12V - charge, J4 Solenoid Power, J5 USB_A, J6 Sel, J7 Conn_01x04, Q1 TIP102, U1 Voltage_regulator_DB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

Commit message: added 3d drawings
Changed lines of the file:
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@@
   (junction (at 99.06 87.63))
   (junction (at 116.205 87.63))
+  (no_connect (at 189.865 36.83))
   (no_connect (at 270.51 156.845))
-  (no_connect (at 189.865 36.83))
   (bus_entry (at 59.69 67.31) (size -2.54 -2.54))
   (bus_entry (at 59.69 69.85) (size -2.54 -2.54))
@@
   (wire (pts (xy 161.29 122.555) (xy 160.02 122.555)))
   (wire (pts (xy 161.29 123.825) (xy 161.29 122.555)))
-  (wire (pts (xy 174.625 122.555) (xy 174.625 128.905)))
+  (wire (pts (xy 174.625 101.6) (xy 178.435 101.6)))
+  (wire (pts (xy 174.625 102.87) (xy 174.625 101.6)))
+  (wire (pts (xy 174.625 121.285) (xy 174.625 128.905)))
   (wire (pts (xy 175.26 108.585) (xy 175.26 109.855)))
   (wire (pts (xy 175.26 109.855) (xy 196.215 109.855)))
-  (wire (pts (xy 175.895 101.6) (xy 178.435 101.6)))
-  (wire (pts (xy 175.895 102.87) (xy 175.895 101.6)))
-  (wire (pts (xy 176.53 123.19) (xy 176.53 133.35)))
+  (wire (pts (xy 176.53 122.555) (xy 176.53 133.35)))
   (wire (pts (xy 178.435 101.6) (xy 178.435 102.235)))
   (wire (pts (xy 178.435 101.6) (xy 183.515 101.6)))
@@
   (wire (pts (xy 184.785 68.58) (xy 186.055 68.58)))
   (wire (pts (xy 184.785 71.755) (xy 209.55 71.755)))
+  (wire (pts (xy 186.055 99.695) (xy 186.055 100.965)))
   (wire (pts (xy 186.055 100.965) (xy 186.055 102.235)))
   (wire (pts (xy 186.055 100.965) (xy 196.215 100.965)))
@@
   (wire (pts (xy 196.85 43.18) (xy 194.31 43.18)))
   (wire (pts (xy 196.85 53.34) (xy 196.85 54.61)))
-  (wire (pts (xy 196.85 123.19) (xy 176.53 123.19)))
-  (wire (pts (xy 196.85 138.43) (xy 196.85 123.19)))
+  (wire (pts (xy 196.85 122.555) (xy 176.53 122.555)))
+  (wire (pts (xy 196.85 138.43) (xy 196.85 122.555)))
   (wire (pts (xy 200.025 62.865) (xy 193.675 62.865)))
   (wire (pts (xy 202.565 128.905) (xy 202.565 133.35)))
@@
   (wire (pts (xy 215.9 113.665) (xy 213.36 113.665)))
   (wire (pts (xy 217.805 128.905) (xy 214.63 128.905)))
-  (wire (pts (xy 219.71 122.555) (xy 174.625 122.555)))
-  (wire (pts (xy 219.71 122.555) (xy 219.71 135.89)))
+  (wire (pts (xy 219.71 121.285) (xy 174.625 121.285)))
+  (wire (pts (xy 219.71 121.285) (xy 219.71 135.89)))
   (wire (pts (xy 219.71 135.89) (xy 217.805 135.89)))
   (bus (pts (xy 57.15 64.77) (xy 57.15 69.85)))
   (bus (pts (xy 57.15 69.85) (xy 57.15 74.93)))
-  (bus (pts (xy 57.15 74.93) (xy 57.15 77.47)))
-  (bus (pts (xy 57.15 77.47) (xy 57.15 87.63)))
+  (bus (pts (xy 57.15 74.93) (xy 57.15 80.01)))
+  (bus (pts (xy 57.15 80.01) (xy 57.15 87.63)))
   (bus (pts (xy 57.15 87.63) (xy 57.15 95.885)))
   (bus (pts (xy 57.15 87.63) (xy 99.06 87.63)))
@@
   (bus (pts (xy 57.15 100.965) (xy 57.15 103.505)))
   (bus (pts (xy 57.15 103.505) (xy 57.15 108.585)))
-  (bus (pts (xy 99.06 62.23) (xy 99.06 67.31)))
-  (bus (pts (xy 99.06 67.31) (xy 99.06 72.39)))
+  (bus (pts (xy 99.06 62.23) (xy 99.06 64.77)))
+  (bus (pts (xy 99.06 64.77) (xy 99.06 69.85)))
+  (bus (pts (xy 99.06 69.85) (xy 99.06 72.39)))
   (bus (pts (xy 99.06 72.39) (xy 99.06 77.47)))
   (bus (pts (xy 99.06 77.47) (xy 99.06 87.63)))
-  (bus (pts (xy 99.06 87.63) (xy 99.06 90.805)))
+  (bus (pts (xy 99.06 87.63) (xy 99.06 93.345)))
   (bus (pts (xy 99.06 87.63) (xy 116.205 87.63)))
-  (bus (pts (xy 99.06 90.805) (xy 99.06 95.885)))
-  (bus (pts (xy 99.06 95.885) (xy 99.06 100.965)))
-  (bus (pts (xy 99.06 100.965) (xy 99.06 106.045)))
-  (bus (pts (xy 99.06 106.045) (xy 99.06 108.585)))
-  (bus (pts (xy 116.205 43.18) (xy 116.205 45.72)))
-  (bus (pts (xy 116.205 45.72) (xy 116.205 63.5)))
-  (bus (pts (xy 116.205 63.5) (xy 116.205 68.58)))
-  (bus (pts (xy 116.205 68.58) (xy 116.205 85.09)))
-  (bus (pts (xy 116.205 85.09) (xy 116.205 87.63)))
+  (bus (pts (xy 99.06 93.345) (xy 99.06 98.425)))
+  (bus (pts (xy 99.06 98.425) (xy 99.06 103.505)))
+  (bus (pts (xy 99.06 103.505) (xy 99.06 108.585)))
+  (bus (pts (xy 116.205 43.18) (xy 116.205 48.26)))
+  (bus (pts (xy 116.205 48.26) (xy 116.205 66.04)))
+  (bus (pts (xy 116.205 66.04) (xy 116.205 82.55)))
+  (bus (pts (xy 116.205 82.55) (xy 116.205 87.63)))
   (bus (pts (xy 116.205 87.63) (xy 116.205 106.045)))
   (bus (pts (xy 116.205 106.045) (xy 116.205 123.825)))
@@
   (bus (pts (xy 157.48 146.05) (xy 167.64 146.05)))
   (bus (pts (xy 157.48 156.21) (xy 157.48 146.05)))
-  (bus (pts (xy 167.64 53.34) (xy 167.64 55.88)))
-  (bus (pts (xy 167.64 55.88) (xy 167.64 76.2)))
-  (bus (pts (xy 167.64 76.2) (xy 167.64 92.71)))
+  (bus (pts (xy 167.64 53.34) (xy 167.64 73.66)))
+  (bus (pts (xy 167.64 73.66) (xy 167.64 92.71)))
   (bus (pts (xy 167.64 92.71) (xy 167.64 113.665)))
   (bus (pts (xy 167.64 113.665) (xy 167.64 133.985)))
@@
     )
   )
-  (symbol (lib_id "power:+12V") (at 186.055 100.965 0) (mirror y) (unit 1)
-    (property "Reference" "#PWR017" (id 0) (at 186.055 104.775 0)
-      (effects (font (size 1.27 1.27)) hide)
-    )
-    (property "Value" "+12V" (id 1) (at 185.674 96.5708 0))
-    (property "Footprint" "" (id 2) (at 186.055 100.965 0)
-      (effects (font (size 1.27 1.27)) hide)
-    )
-    (property "Datasheet" "" (id 3) (at 186.055 100.965 0)
+  (symbol (lib_id "power:+12V") (at 186.055 99.695 0) (mirror y) (unit 1)
+    (property "Reference" "#PWR017" (id 0) (at 186.055 103.505 0)
+      (effects (font (size 1.27 1.27)) hide)
+    )
+    (property "Value" "+12V" (id 1) (at 185.674 95.3008 0))
+    (property "Footprint" "" (id 2) (at 186.055 99.695 0)
+      (effects (font (size 1.27 1.27)) hide)
+    )
+    (property "Datasheet" "" (id 3) (at 186.055 99.695 0)
       (effects (font (size 1.27 1.27)) hide)
     )
@@
     )
   )
-  (symbol (lib_id "power:GNDREF") (at 175.895 102.87 0) (mirror y) (unit 1)
-    (property "Reference" "#PWR0105" (id 0) (at 175.895 109.22 0)
-      (effects (font (size 1.27 1.27)) hide)
-    )
-    (property "Value" "GNDREF" (id 1) (at 175.895 106.68 0)
-      (effects (font (size 1.27 1.27)) hide)
-    )
-    (property "Footprint" "" (id 2) (at 175.895 102.87 0)
-      (effects (font (size 1.27 1.27)) hide)
-    )
-    (property "Datasheet" "" (id 3) (at 175.895 102.87 0)
-      (effects (font (size 1.27 1.27)) hide)
-    )
+  (symbol (lib_id "power:GNDREF") (at 174.625 102.87 0) (mirror y) (unit 1)
+    (property "Reference" "#PWR0105" (id 0) (at 174.625 109.22 0)
+      (effects (font (size 1.27 1.27)) hide)
+    )
+    (property "Value" "GNDREF" (id 1) (at 174.625 106.68 0)
+      (effects (font (size 1.27 1.27)) hide)
+    )
+    (property "Footprint" "" (id 2) (at 174.625 102.87 0)
+      (effects (font (size 1.27 1.27)) hide)
+    )
+    (property "Datasheet" "" (id 3) (at 174.625 102.87 0)
+      (effects (font (size 1.27 1.27)) hide)
+    )
