File: SlugCharge Motherboard/KiCad Project Files/UI.kicad_pcb (KiCad board)
At the start: 2 copper layers, 120 x 120 mm, 66 parts, among them J1 16x2 LCD Display, J10 Speaker, J12 , J2 RAW in, J3 3x4 Keypad, J4 Conn_02x03_Odd_Even, J5 Locker4-6, J6 Locker1-3, P1 USB_C_Plug, SW1 RST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

Commit message: added 3d drawings
Parts:
- added C13: 100nF, Capacitor_SMD:C_0805_2012Metric_Pad1.15x1.40mm_HandSolder, F.Cu at (117.0, 99.5)
- added C19: 100nF, Capacitor_SMD:C_0805_2012Metric_Pad1.15x1.40mm_HandSolder, F.Cu at (116.5, 108.5)
- added C20: 100nF, Capacitor_SMD:C_0805_2012Metric_Pad1.15x1.40mm_HandSolder, F.Cu at (67.5, 71.0)
- added C21: 100nF, Capacitor_SMD:C_0805_2012Metric_Pad1.15x1.40mm_HandSolder, F.Cu at (114.5, 108.5)
- added D1: LED_Small, Connector_PinHeader_2.54mm:PinHeader_1x02_P2.54mm_Vertical, F.Cu at (130.5, 103.0)
- added Q1: IRF520, Package_TO_SOT_THT:TO-220-3_Vertical, F.Cu at (122.5, 110.1)
- added R15: 300K, Resistor_SMD:R_0805_2012Metric, F.Cu at (118.5, 104.1)
- added R16: 20K, Resistor_SMD:R_0805_2012Metric, F.Cu at (110.6, 105.5)
- added R17: 100K, Resistor_SMD:R_0805_2012Metric, F.Cu at (118.5, 108.4)
- added R18: 400K, Resistor_SMD:R_0805_2012Metric, F.Cu at (110.6, 102.5)
- added R19: 32.4K, Resistor_SMD:R_0805_2012Metric, F.Cu at (112.0, 108.4)
- added R7: 510R, Resistor_SMD:R_0805_2012Metric, F.Cu at (128.0, 106.5)
- added R8: 10K, Resistor_SMD:R_0805_2012Metric, F.Cu at (113.6, 100.0)
- added U1: TLV3201, Package_TO_SOT_SMD:SOT-23-5, F.Cu at (115.0, 104.1)
- D3, D4: value D_Schottky -> 1N4004
- J12: value (none) -> Power
- J4: value Conn_02x03_Odd_Even -> ICSP
- R1: value 1KΩ -> 10KΩ
Connections:
- net Net-(C10-Pad1) renamed /OSC2
- net Net-(C12-Pad1) renamed /AREF
- net Net-(C9-Pad1) renamed /OSC1
- C1 pad 2: GNDREF -> +5V
- C10 pad 2: GNDREF -> +5V
- C11 pad 2: GNDREF -> +5V
- C12 pad 2: GNDREF -> +5V
- C14 pad 1: GNDREF -> +5V
- C15 pad 1: GNDREF -> +5V
- C17 pad 2: GNDREF -> +5V
- C18 pad 2: GNDREF -> +5V
- C2 pad 1: GNDREF -> +5V
- C3 pad 1: GNDREF -> +5V
- C37 pad 1: GNDREF -> +5V
- C4 pad 2: GNDREF -> +5V
- C5 pad 1: GNDREF -> +5V
- C50 pad 2: GNDREF -> +5V
- C51 pad 2: GNDREF -> +5V
- C52 pad 2: GNDREF -> +5V
- C6 pad 1: GNDREF -> +5V
- C7 pad 2: GNDREF -> +5V
- C8 pad 2: GNDREF -> +5V
- C9 pad 2: GNDREF -> +5V
- D13 pad 1: GNDREF -> +5V
- J1 pad 1: GNDREF -> +5V
- J1 pad 16: GNDREF -> +5V
- J1 pad 5: GNDREF -> +5V
- J12 pad 1: GNDREF -> +5V
- J12 pad 2: +VSW -> +BATT
- J12 pad 3: GNDREF -> +5V
- J12 pad 4: +VSW -> +BATT
- J12 pad 5: GNDREF -> +5V
- J2 pad 1: GNDREF -> +5V
- J2 pad 2: +VSW -> +BATT
- J2 pad 3: GNDREF -> +5V
- J2 pad 4: +VSW -> +BATT
- J4 pad 6: GNDREF -> +5V
- PWR1 pad 1: GNDREF -> +5V
- R11 pad 2: +VSW -> +BATT
- R12 pad 1: GNDREF -> +5V
- R13 pad 2: +VSW -> +BATT
- R14 pad 1: GNDREF -> +5V
- R3 pad 2: GNDREF -> +5V
- R6 pad 2: GNDREF -> +5V
- RV1 pad 3: GNDREF -> +5V
- SW1 pad 2: GNDREF -> +5V
- U2 pad 1: GNDREF -> +5V
- U3 pad 1: GNDREF -> +5V
- U3 pad 5: /D+ -> /Programming/Interrupt(subsheet)/D+
- U3 pad 6: /D- -> /Programming/Interrupt(subsheet)/D-
- U4 pad 11: GNDREF -> +5V
- U4 pad 32: GNDREF -> +5V
- U4 pad 62: GNDREF -> +5V
- U4 pad 81: GNDREF -> +5V
- U4 pad 97: Net-(U4-Pad97) -> /BLI
- U4 pad 99: GNDREF -> +5V
- U5 pad 7: GNDREF -> +5V
- Y1 pad 2: GNDREF -> +5V
- Y1 pad 4: GNDREF -> +5V
- Y2 pad 2: GNDREF -> +5V
- Y2 pad 4: GNDREF -> +5V
Routing:
- net /BLI: track 0.00 -> 80.4 mm, vias 0 -> 1
- net +5V: track 46.9 -> 91.5 mm, vias 10 -> 60
- net GNDREF: track 41.8 -> 3.35 mm, vias 48 -> 0
- net +BATT: track 0.00 -> 18.1 mm, vias 0 -> 82
- net Net-(D1-Pad1): track 0.00 -> 12.1 mm
- net Net-(C21-Pad1): track 0.00 -> 11.1 mm
- net Net-(C19-Pad1): track 0.00 -> 7.03 mm
- net Net-(R18-Pad2): track 0.00 -> 5.62 mm
- net Net-(D1-Pad2): track 0.00 -> 2.51 mm
- net /Programming/Interrupt(subsheet)/D+: vias 0 -> 2
- net /D+: vias 2 -> 0
- net +VSW: vias 82 -> 0
- added copper zone on B.Cu, net +5V
- added copper zone on B.Cu, net +BATT
- added copper zone on F.Cu, net +BATT
- removed copper zone on B.Cu, net +VSW
- removed copper zone on F.Cu, net +VSW
- removed copper zone on B.Cu, net GNDREF
- removed copper zone on F.Cu, net GNDREF
