File: SlugCharge Motherboard/KiCad Project Files/UI.kicad_sch (KiCad schematic)
At the start: 33 parts, among them J1 16x2 LCD Display, J10 Speaker, J12 Power, J2 RAW in, J5 Locker4-6, J6 Locker1-3, U2 ams1117-3.3V, U4 ATmega2560-16AU

Commit message: added 3d drawings
Parts:
- U4: symbol Custom_Symbols:AtMega2560 -> Custom_Symbols_new:AtMega2560
Connections:
- net Programming/Interrupt(subsheet)/BLI: now reaches U4.97 (PF0)
- net +VSW renamed +BATT
- no-connect marks 42 -> 41
Other:
- sheet Programming/Interrupt(subsheet) ports: added BLI; removed none
- note added: "Battery Low Interrupt"
